Commit message: introduced xacro macros to enable reusability of the open manipulator pro URDF

File: open_manipulator_p_description/urdf/open_manipulator_p_with_gripper.urdf.xacro (robot description, xacro)
@@ -2,346 +2,10 @@
 <!-- Revolute-Revolute Manipulator -->
 <robot name="open_manipulator_p" xmlns:xacro="http://www.ros.org/wiki/xacro">
-  <!-- some parameters -->
-  <xacro:property name="pi" value="3.141592654" />
-  <!-- some parameters -->
-  <xacro:property name="pi" value="3.141592654" />
   <!-- Import all Gazebo-customization elements, including Gazebo colors -->
-  <xacro:include filename="$(find open_manipulator_p_description)/urdf/open_manipulator_p_with_gripper.gazebo.xacro" />
-  <!-- Import Rviz colors -->
-  <xacro:include filename="$(find open_manipulator_p_description)/urdf/materials.xacro" />
-  <!-- Transmission macro -->
-  <xacro:macro name="SimpleTransmission" params="joint n">
-    <transmission name="tran${n}">
-      <type>transmission_interface/SimpleTransmission</type>
-      <joint name="${joint}">
-        <hardwareInterface>hardware_interface/PositionJointInterface</hardwareInterface>
-      </joint>
-      <actuator name="motor${n}">
-        <hardwareInterface>hardware_interface/PositionJointInterface</hardwareInterface>
-        <mechanicalReduction>1</mechanicalReduction>
-      </actuator>
-    </transmission>
-  </xacro:macro>
+  <xacro:include filename="$(find open_manipulator_p_description)/urdf/open_manipulator_p_with_gripper_macro.urdf.xacro"/>
   <!-- World -->
-  <link name="world">
-  </link>
-  <!-- World fixed joint-->
-  <joint name="world_fixed" type="fixed">
-    <origin xyz="0 0 0" rpy="0 0 0"/>
-    <parent link="world"/>
-    <child link="link1"/>
-  </joint>
-  <!-- link 1 -->
-  <link name="link1">
-    <collision>
-      <origin xyz="0 0 0" rpy="0 0 0"/>
-      <geometry>
-        <mesh filename="package://open_manipulator_p_description/meshes/link_1.stl" scale="0.001 0.001 0.001"/>
-      </geometry>
-    </collision>
-    <visual>
-      <origin xyz="0 0 0" rpy="0 0 0"/>
-      <geometry>
-        <mesh filename="package://open_manipulator_p_description/meshes/link_1.stl" scale="0.001 0.001 0.001"/>
-      </geometry>
-      <material name="grey"/>
-    </visual>
-    <inertial>
-      <origin xyz="0.00023 0.00000 0.06223" rpy="0 0 0"/>
-      <mass value="0.85644"/>
-      <inertia ixx="1.0" ixy="0.0" ixz="0.0" iyy="1.0" iyz="0.0" izz="1.0" />
-      <!--<inertia ixx="0.00121064" ixy="0.0" ixz="0.00001100" iyy="0.00120886" iyz="0.0" izz="0.00038103" />-->
-    </inertial>
-  </link>
-  <!-- Joint 1 -->
-  <joint name="joint1" type="revolute">
-    <parent link="link1"/>
-    <child link="link2"/>
-    <origin xyz="0.0 0.0 0.126" rpy="0 0 0"/>
-    <axis xyz="0 0 1"/>
-    <limit velocity="6.5" effort="1000" lower="${-pi*0.5}" upper="${pi*0.5}" />
-    <dynamics damping="0.7"/>
-  </joint>
-  <!-- Transmission 1 -->
-  <xacro:SimpleTransmission n="1" joint="joint1" />
-  <!-- link 2 -->
-  <link name="link2">
-    <collision>
-      <origin xyz="0 0 0" rpy="0 0 0"/>
-      <geometry>
-        <mesh filename="package://open_manipulator_p_description/meshes/link_2.stl" scale="0.001 0.001 0.001"/>
-      </geometry>
-    </collision>
-    <visual>
-      <origin xyz="0 0 0" rpy="0 0 0"/>
-      <geometry>
-        <mesh filename="package://open_manipulator_p_description/meshes/link_2.stl" scale="0.001 0.001 0.001"/>
-      </geometry>
-      <material name="grey"/>
-    </visual>
-    <inertial>
-      <origin xyz="0.00000 0.00080 0.03183" rpy="0 0 0"/>
-      <!--<origin xyz="0.00000 -0.06820 -0.00117" rpy="0 0 0"/>-->
-      <mass value="0.94658"/>
-      <inertia ixx="1.0" ixy="0.0" ixz="0.0" iyy="1.0" iyz="0.0" izz="1.0" />
-      <!--<inertia ixx="0.00152547" ixy="0.0" ixz="0.0" iyy="0.00045954" iyz="-0.00001086" izz="0.00151740" />-->
-    </inertial>
-  </link>
-  <!-- Joint 2 -->
-  <joint name="joint2" type="revolute">
-    <parent link="link2"/>
-    <child link="link3"/>
-    <origin xyz="0.0 0.069 0.033" rpy="0 0 0"/>
-    <axis xyz="0 1 0"/>
-    <limit velocity="6.5" effort="1000" lower="${-pi*0.5}" upper="${pi*0.5}" />
-    <dynamics damping="0.7"/>
-  </joint>
-  <!-- Transmission 2 -->
-  <xacro:SimpleTransmission n="2" joint="joint2" />
-  <!-- link 3 -->
-  <link name="link3">
-    <collision>
-      <origin xyz="0 0 0" rpy="0 0 0"/>
-      <geometry>
-        <mesh filename="package://open_manipulator_p_description/meshes/link_3.stl" scale="0.001 0.001 0.001"/>
-      </geometry>
-    </collision>
-    <visual>
-      <origin xyz="0 0 0" rpy="0 0 0"/>
-      <geometry>
-        <mesh filename="package://open_manipulator_p_description/meshes/link_3.stl" scale="0.001 0.001 0.001"/>
-      </geometry>
-      <material name="grey"/>
-    </visual>
-    <inertial>
-      <origin xyz="0.01768 -0.06881 0.20524" rpy="0 0 0"/>
-      <!--<origin xyz="-0.01232 -0.05731 -0.05876" rpy="0 0 0"/>-->
-      <mass value="1.30260"/>
-      <inertia ixx="1.0" ixy="0.0" ixz="0.0" iyy="1.0" iyz="0.0" izz="1.0" />
-      <!--<inertia ixx="0.01111021" ixy="0.00001331" ixz="-0.00134208" iyy="0.01046642" iyz="0.00016235" izz="0.00202081" />-->
-    </inertial>
-  </link>
-  <!-- Joint 3 -->
-  <joint name="joint3" type="revolute">
-    <parent link="link3"/>
-    <child link="link4"/>
-    <origin xyz="0.03000 -0.01150 0.26400" rpy="0 0 0"/>
-    <axis xyz="0 1 0"/>
-    <limit velocity="6.5" effort="1000" lower="${-pi*0.5}" upper="${pi*0.5}" />
-    <dynamics damping="0.7"/>
-  </joint>
-  <!-- Transmission 3 -->
-  <xacro:SimpleTransmission n="3" joint="joint3" />
-  <!-- link 4 -->
-  <link name="link4">
-    <collision>
-      <origin xyz="0 0 0" rpy="0 0 0"/>
-      <geometry>
-        <mesh filename="package://open_manipulator_p_description/meshes/link_4.stl" scale="0.001 0.001 0.001"/>
-      </geometry>
-    </collision>
-    <visual>
-      <origin xyz="0 0 0" rpy="0 0 0"/>
-      <geometry>
-        <mesh filename="package://open_manipulator_p_description/meshes/link_4.stl" scale="0.001 0.001 0.001"/>
-      </geometry>
-      <material name="grey"/>
-    </visual>
-    <inertial>
-      <origin xyz="0.12475 -0.05716 0.02979" rpy="0 0 0"/>
-      <!--<origin xyz="-0.07025 0.00034 -0.00021" rpy="0 0 0"/>-->
-      <mass value="1.15977"/>
-      <inertia ixx="1.0" ixy="0.0" ixz="0.0" iyy="1.0" iyz="0.0" izz="1.0" />
-      <!--<inertia ixx="0.00096726" ixy="0.00004383" ixz="-0.00002771" iyy="0.00318801" iyz="0.00000627" izz="0.00341484" />-->
-    </inertial>
-  </link>
-  <!-- Joint 4 -->
-  <joint name="joint4" type="revolute">
-    <parent link="link4"/>
-    <child link="link5"/>
-    <origin xyz="0.19500 -0.05750 0.03000" rpy="0 0 0"/>
-    <axis xyz="1 0 0"/>
-    <limit velocity="6.5" effort="1000" lower="${-pi*0.5}" upper="${pi*0.5}" />
-    <dynamics damping="0.7"/>
-  </joint>
-  <!-- Transmission 4 -->
-  <xacro:SimpleTransmission n="4" joint="joint4" />
-  <!-- link 5 -->
-  <link name="link5">
-    <collision>
-      <origin xyz="0 0 0" rpy="0 0 0"/>
-      <geometry>
-        <mesh filename="package://open_manipulator_p_description/meshes/link_5.stl" scale="0.001 0.001 0.001"/>
-      </geometry>
-    </collision>
-    <visual>
-      <origin xyz="0 0 0" rpy="0 0 0"/>
-      <geometry>
-        <mesh filename="package://open_manipulator_p_description/meshes/link_5.stl" scale="0.001 0.001 0.001"/>
-      </geometry>
-      <material name="grey"/>
-    </visual>
-    <inertial>
-      <origin xyz="0.05642 -0.00217 0.00002" rpy="0 0 0"/>
-      <!--<origin xyz="-0.00658 -0.04717 0.00002" rpy="0 0 0"/>-->
-      <mass value="0.44688"/>
-      <inertia ixx="1.0" ixy="0.0" ixz="0.0" iyy="1.0" iyz="0.0" izz="1.0" />
-      <!--<inertia ixx="0.00030285" ixy="0.00000761" ixz="0.00000031" iyy="0.00022339" iyz="-0.00000001" izz="0.00039766" />-->
-    </inertial>
-  </link>
-  <!-- Joint 5 -->
-  <joint name="joint5" type="revolute">
-    <parent link="link5"/>
-    <child link="link6"/>
-    <origin xyz="0.06300 0.04500 0.00000" rpy="0 0 0"/>
-    <axis xyz="0 1 0"/>
-    <limit velocity="6.5" effort="1000" lower="${-pi*0.5}" upper="${pi*0.5}" />
-    <dynamics damping="0.7"/>
-  </joint>
-  <!-- Transmission 5 -->
-  <xacro:SimpleTransmission n="5" joint="joint5" />
-  <!-- link 6 -->
-  <link name="link6">
-    <collision>
-      <origin xyz="0 0 0" rpy="0 0 0"/>
-      <geometry>
-        <mesh filename="package://open_manipulator_p_description/meshes/link_6.stl" scale="0.001 0.001 0.001"/>
-      </geometry>
-    </collision>
-    <visual>
-      <origin xyz="0 0 0" rpy="0 0 0"/>
-      <geometry>
-        <mesh filename="package://open_manipulator_p_description/meshes/link_6.stl" scale="0.001 0.001 0.001"/>
-      </geometry>
-      <material name="grey"/>
-    </visual>
-    <inertial>
-      <origin xyz="0.06831 -0.04457 0.00000" rpy="0 0 0"/>
-      <!--<origin xyz="-0.05469 0.00043 0.00000" rpy="0 0 0"/>-->
-      <mass value="0.43273"/>
-      <inertia ixx="1.0" ixy="0.0" ixz="0.0" iyy="1.0" iyz="0.0" izz="1.0" />
-      <!--<inertia ixx="0.00021512" ixy="0.00001009" ixz="0.00000000" iyy="0.00042827" iyz="0.00000000" izz="0.00051436" />-->
-    </inertial>
-  </link>
-  <!-- Joint 6 -->
-  <joint name="joint6" type="revolute">
-    <parent link="link6"/>
-    <child link="gripper_main_link"/>
-    <origin xyz="0.12300 -0.04500 0.00000" rpy="0 0 0"/>
-    <axis xyz="1 0 0"/>
-    <limit velocity="6.5" effort="1000" lower="${-pi*0.5}" upper="${pi*0.5}" />
-    <dynamics damping="0.7"/>
-  </joint>
-  <!-- Transmission 6 -->
-  <xacro:SimpleTransmission n="6" joint="joint6" />
-  <!-- gripper main link -->
-  <link name="gripper_main_link">
-    <collision>
-      <origin xyz="0 0 0" rpy="0 0 0" />
-      <geometry>
-        <mesh filename="package://open_manipulator_p_description/meshes/gripper_main_link.stl" scale="0.001 0.001 0.001"/>
-      </geometry>
-    </collision>
-    <visual>
-      <origin xyz="0 0 0" rpy="0 0 0" />
-      <geometry>
-        <mesh filename="package://open_manipulator_p_description/meshes/gripper_main_link.stl" scale="0.001 0.001 0.001"/>
-      </geometry>
-      <material name="grey"/>
-    </visual>
-    <inertial>
-      <origin xyz="0.0 0.0 0.0" rpy="0 0 0"/>
-      <mass value="0.509"/>
-      <inertia ixx="1.0" ixy="0.0" ixz="0.0" iyy="1.0" iyz="0.0" izz="1.0" />
-    </inertial>
-  </link>
-  <!-- gripper joint -->
-  <joint name="gripper" type="revolute">
-    <axis xyz="0 0 -1" />
-    <origin xyz="0.0552 -0.0460 0" rpy="0 0 ${45.0*pi/180.0}"/>
-    <!-- <origin xyz="0.0552 -0.0370 0" rpy="0 0 0"/> -->
-    <parent link="gripper_main_link"/>
-    <child link="gripper_link"/>
-    <limit velocity="6.5" effort="1000" lower="0.0" upper="${740.0/2048.0*pi}" />
-    <dynamics damping="0.1" friction="0.0" />
-  </joint>
-  <!-- Transmission gripper -->
-  <xacro:SimpleTransmission n="_gripper" joint="gripper" />
-  <!-- gripper link -->
-  <link name="gripper_link">
-    <collision>
-      <origin xyz="0 0 0" rpy="0 0 0" />
-      <geometry>
-        <mesh filename="package://open_manipulator_p_description/meshes/gripper_link.stl" scale="0.001 0.001 0.001"/>
-      </geometry>
-      <material name="grey"/>
-    </collision>
-    <visual>
-      <origin xyz="0 0 0" rpy="0 0 0" />
-      <geometry>
-        <mesh filename="package://open_manipulator_p_description/meshes/gripper_link.stl" scale="0.001 0.001 0.001"/>
-      </geometry>
-      <material name="grey"/>
-    </visual>
-    <inertial>
-      <origin xyz="0 0 0" rpy="0 0 0"/>
-      <mass value="0.013"/>
-      <inertia ixx="1.0" ixy="0.0" ixz="0.0" iyy="1.0" iyz="0.0" izz="1.0" />
-    </inertial>
-  </link>
-  <!-- gripper joint 1 -->
-  <joint name="gripper_sub" type="revolute">
-    <axis xyz="0 0 1" />
-    <origin xyz="0.0552 0.0460 0" rpy="0 0 ${-45.0*pi/180.0}"/>
-    <!-- <origin xyz="0.0552 0.0370 0" rpy="0 0 0"/> -->
-    <parent link="gripper_main_link"/>
-    <child link="gripper_sub_link"/>
-    <limit velocity="6.5" effort="1000" lower="0.0" upper="${740.0/2048.0*pi}" />
-    <dynamics damping="0.1" friction="0.0" />
-  </joint>
-  <!-- Transmission gripper -->
-  <xacro:SimpleTransmission n="_gripper_sub" joint="gripper_sub" />
-  <!-- gripper 1 link -->
-  <link name="gripper_sub_link">
-    <collision>
-      <origin xyz="0 0 0" rpy="0 0 0" />
-      <geometry>
-        <mesh filename="package://open_manipulator_p_description/meshes/gripper_sub_link.stl" scale="0.001 0.001 0.001"/>
-      </geometry>
-      <material name="grey"/>
-    </collision>
-    <visual>
-      <origin xyz="0 0 0" rpy="0 0 0" />
-      <geometry>
-        <mesh filename="package://open_manipulator_p_description/meshes/gripper_sub_link.stl" scale="0.001 0.001 0.001"/>
-      </geometry>
-      <material name="grey"/>
-    </visual>
-    <inertial>
-      <origin xyz="0 0 0" rpy="0 0 0"/>
-      <mass value="0.013"/>
-      <inertia ixx="1.0" ixy="0.0" ixz="0.0" iyy="1.0" iyz="0.0" izz="1.0" />
-    </inertial>
-  </link>
-  <!-- gripper main fixed joint-->
-  <joint name="gripper_main_fixed" type="fixed">
-    <parent link="gripper_main_link"/>
-    <child link="end_effector"/>
-    <origin xyz="0.14 0.0 0.0" rpy="0 0 0" />
-  </joint>
-  <!-- End Effector -->
-  <link name="end_effector">
-    <visual>
-      <origin xyz="0.0 0.0 0.0" rpy="0 0 0" />
-      <geometry>
-        <box size = "0.01 0.01 0.01"/>
-      </geometry>
-      <material name="red"/>
-    </visual>
-    <inertial>
-      <origin xyz="0.0 0.0 0.0" rpy="0 0 0" />
-      <mass value="0.001" />
-      <inertia ixx="1.0" ixy="0.0" ixz="0.0" iyy="1.0" iyz="0.0" izz="1.0" />
-    </inertial>
-  </link>
+  <link name="world"></link>
+  <xacro:open_manipulator_p_with_gripper_macro parent="world" name="arm">
+    <origin xyz="0.0 0.0 0.0" rpy="0 0 0"/>
+  </xacro:open_manipulator_p_with_gripper_macro>
 </robot>

Commit message: added ros controllers

File: open_manipulator_p_description/urdf/open_manipulator_p.gazebo.xacro (robot description, xacro)
@@ -2,9 +2,10 @@
 <robot xmlns:xacro="http://www.ros.org/wiki/xacro">
   <xacro:macro name="open_manipulator_p_gazebo_macro" params="name">
-    <!-- ros_control plugin -->
+    <!-- Gazebo ros control for arm joints -->
     <gazebo>
-      <plugin name="gazebo_ros_control" filename="libgazebo_ros_control.so">
-        <robotNamespace>open_manipulator_p</robotNamespace>
-        <robotSimType>gazebo_ros_control/DefaultRobotHWSim</robotSimType>
+      <plugin name="gazebo_ros_control_select_joints" filename="libgazebo_ros_control_select_joints.so">
+        <robotNamespace>manipulator_arm_control</robotNamespace>
+        <joints>${name}_joint1 ${name}_joint2 ${name}_joint3 ${name}_joint4 ${name}_joint5 ${name}_joint6 ${name}_gripper ${name}_gripper_sub</joints>
+        <eStopTopic>/ui_emergency_stop</eStopTopic>
       </plugin>
     </gazebo>
@@ -13,5 +14,5 @@
       <mu1>0.2</mu1>
       <mu2>0.2</mu2>
-      <material>Gazebo/Grey</material>
+      <material>Gazebo/DarkGrey</material>
     </gazebo>
     <!-- Link2 -->
@@ -19,5 +20,5 @@
       <mu1>0.2</mu1>
       <mu2>0.2</mu2>
-      <material>Gazebo/Grey</material>
+      <material>Gazebo/DarkGrey</material>
     </gazebo>
     <!-- Link3 -->
@@ -25,5 +26,5 @@
       <mu1>0.2</mu1>
       <mu2>0.2</mu2>
-      <material>Gazebo/Grey</material>
+      <material>Gazebo/DarkGrey</material>
     </gazebo>
     <!-- Link4 -->
@@ -31,5 +32,5 @@
       <mu1>0.2</mu1>
       <mu2>0.2</mu2>
-      <material>Gazebo/Grey</material>
+      <material>Gazebo/DarkGrey</material>
     </gazebo>
     <!-- Link5 -->
@@ -37,5 +38,5 @@
       <mu1>0.2</mu1>
       <mu2>0.2</mu2>
-      <material>Gazebo/Grey</material>
+      <material>Gazebo/DarkGrey</material>
     </gazebo>
     <!-- Link6 -->
@@ -43,5 +44,5 @@
       <mu1>0.2</mu1>
       <mu2>0.2</mu2>
-      <material>Gazebo/Grey</material>
+      <material>Gazebo/DarkGrey</material>
     </gazebo>
     <!-- End Effector -->
@@ -49,5 +50,5 @@
       <mu1>0.2</mu1>
       <mu2>0.2</mu2>
-      <material>Gazebo/Grey</material>
+      <material>Gazebo/DarkGrey</material>
     </gazebo>
   </xacro:macro>

File: open_manipulator_p_description/urdf/open_manipulator_p_macro.urdf.xacro (robot description, xacro)
@@ -20,4 +20,5 @@
   </xacro:macro>
   <xacro:macro name="open_manipulator_p_macro" params="name parent *origin">
+    <xacro:open_manipulator_p_gazebo_macro name="${name}"/>
     <joint name="${name}_fixed_joint" type="fixed">
       <xacro:insert_block name="origin"/>

File: open_manipulator_p_description/urdf/open_manipulator_p_with_gripper.gazebo.xacro (robot description, xacro)
@@ -3,10 +3,9 @@
   <xacro:include filename="$(find open_manipulator_p_description)/urdf/open_manipulator_p.gazebo.xacro"/>
   <xacro:macro name="open_manipulator_p_with_gripper_gazebo_macro" params="name">
-    <xacro:open_manipulator_p_gazebo_macro name="${name}"/>
     <!-- gripper main link -->
     <gazebo reference="${name}_gripper_main_link">
       <mu1>0.2</mu1>
       <mu2>0.2</mu2>
-      <material>Gazebo/Grey</material>
+      <material>Gazebo/DarkGrey</material>
     </gazebo>
     <!-- gripper link -->
@@ -14,5 +13,5 @@
       <mu1>0.2</mu1>
       <mu2>0.2</mu2>
-      <material>Gazebo/Grey</material>
+      <material>Gazebo/DarkGrey</material>
     </gazebo>
     <!-- gripper 1 link -->
@@ -20,5 +19,5 @@
       <mu1>0.2</mu1>
       <mu2>0.2</mu2>
-      <material>Gazebo/Grey</material>
+      <material>Gazebo/DarkGrey</material>
     </gazebo>
     <!-- End Effector -->
