Commit message: adjusted the joint and link naming scheme to match our other robots

File: open_manipulator_p_description/urdf/open_manipulator_p.gazebo.xacro (robot description, xacro)
@@ -6,40 +6,40 @@
       <plugin name="gazebo_ros_control_select_joints" filename="libgazebo_ros_control_select_joints.so">
         <robotNamespace>manipulator_arm_control</robotNamespace>
-        <joints>${name}_joint1 ${name}_joint2 ${name}_joint3 ${name}_joint4 ${name}_joint5 ${name}_joint6 ${name}_gripper ${name}_gripper_sub</joints>
+        <joints>${name}_joint_0 ${name}_joint_1 ${name}_joint_2 ${name}_joint_3 ${name}_joint_4 ${name}_joint_5 ${name}_gripper ${name}_gripper_sub</joints>
         <eStopTopic>/ui_emergency_stop</eStopTopic>
       </plugin>
     </gazebo>
-    <!-- Link1 -->
-    <gazebo reference="${name}_link1">
+    <!-- Link 0 -->
+    <gazebo reference="${name}_link_0">
       <mu1>0.2</mu1>
       <mu2>0.2</mu2>
       <material>Gazebo/DarkGrey</material>
     </gazebo>
-    <!-- Link2 -->
-    <gazebo reference="${name}_link2">
+    <!-- Link 1 -->
+    <gazebo reference="${name}_link_1">
       <mu1>0.2</mu1>
       <mu2>0.2</mu2>
       <material>Gazebo/DarkGrey</material>
     </gazebo>
-    <!-- Link3 -->
-    <gazebo reference="${name}_link3">
+    <!-- Link 2 -->
+    <gazebo reference="${name}_link_2">
       <mu1>0.2</mu1>
       <mu2>0.2</mu2>
       <material>Gazebo/DarkGrey</material>
     </gazebo>
-    <!-- Link4 -->
-    <gazebo reference="${name}_link4">
+    <!-- Link 3 -->
+    <gazebo reference="${name}_link_3">
       <mu1>0.2</mu1>
       <mu2>0.2</mu2>
       <material>Gazebo/DarkGrey</material>
     </gazebo>
-    <!-- Link5 -->
-    <gazebo reference="${name}_link5">
+    <!-- Link 4 -->
+    <gazebo reference="${name}_link_4">
       <mu1>0.2</mu1>
       <mu2>0.2</mu2>
       <material>Gazebo/DarkGrey</material>
     </gazebo>
-    <!-- Link6 -->
-    <gazebo reference="${name}_link6">
+    <!-- Link 5 -->
+    <gazebo reference="${name}_link_5">
       <mu1>0.2</mu1>
       <mu2>0.2</mu2>

File: open_manipulator_p_description/urdf/open_manipulator_p_macro.urdf.xacro (robot description, xacro)
@@ -24,13 +24,8 @@
       <xacro:insert_block name="origin"/>
       <parent link="${parent}"/>
-      <child link="${name}_mount_link"/>
-    </joint>
-    <link name="${name}_mount_link"></link>
-    <joint name="${name}_joint0" type="fixed">
-      <parent link="${name}_mount_link"/>
-      <child link="${name}_link1"/>
-    </joint>
-    <!-- link 1 -->
-    <link name="${name}_link1">
+      <child link="${name}_link_0"/>
+    </joint>
+    <!-- link 0 -->
+    <link name="${name}_link_0">
       <collision>
         <origin xyz="0 0 0.063" rpy="0 0 0" />
@@ -53,8 +48,8 @@
       </inertial>
     </link>
-    <!-- Joint 1 -->
-    <joint name="${name}_joint1" type="revolute">
-      <parent link="${name}_link1"/>
-      <child link="${name}_link2"/>
+    <!-- Joint 0 -->
+    <joint name="${name}_joint_0" type="revolute">
+      <parent link="${name}_link_0"/>
+      <child link="${name}_link_1"/>
       <origin xyz="0.0 0.0 0.126" rpy="0 0 0"/>
       <axis xyz="0 0 1"/>
@@ -62,8 +57,8 @@
       <dynamics damping="0.7"/>
     </joint>
-    <!-- Transmission 1 -->
-    <xacro:SimpleTransmission n="1" joint="${name}_joint1"/>
-    <!-- link 2 -->
-    <link name="${name}_link2">
+    <!-- Transmission 0 -->
+    <xacro:SimpleTransmission n="0" joint="${name}_joint_0"/>
+    <!-- link 1 -->
+    <link name="${name}_link_1">
       <collision>
         <origin xyz="0 0 0.03" rpy="0 0 0" />
@@ -87,8 +82,8 @@
       </inertial>
     </link>
-    <!-- Joint 2 -->
-    <joint name="${name}_joint2" type="revolute">
-      <parent link="${name}_link2"/>
-      <child link="${name}_link3"/>
+    <!-- Joint 1 -->
+    <joint name="${name}_joint_1" type="revolute">
+      <parent link="${name}_link_1"/>
+      <child link="${name}_link_2"/>
       <origin xyz="0.0 0.0 0.033" rpy="0 0 0"/>
       <axis xyz="0 1 0"/>
@@ -96,8 +91,8 @@
       <dynamics damping="0.7"/>
     </joint>
-    <!-- Transmission 2 -->
-    <xacro:SimpleTransmission n="2" joint="${name}_joint2"/>
-    <!-- link 3 -->
-    <link name="${name}_link3">
+    <!-- Transmission 1 -->
+    <xacro:SimpleTransmission n="1" joint="${name}_joint_1"/>
+    <!-- link 2 -->
+    <link name="${name}_link_2">
       <collision>
         <origin xyz="0.0 0.07 0.01" rpy="0 0 0" />
@@ -144,8 +139,8 @@
       </inertial>
     </link>
-    <!-- Joint 3 -->
-    <joint name="${name}_joint3" type="revolute">
-      <parent link="${name}_link3"/>
-      <child link="${name}_link4"/>
+    <!-- Joint 2 -->
+    <joint name="${name}_joint_2" type="revolute">
+      <parent link="${name}_link_2"/>
+      <child link="${name}_link_3"/>
       <origin xyz="0.03000 0.0 0.26400" rpy="0 0 0"/>
       <axis xyz="0 1 0"/>
@@ -153,8 +148,8 @@
       <dynamics damping="0.7"/>
     </joint>
-    <!-- Transmission 3 -->
-    <xacro:SimpleTransmission n="3" joint="${name}_joint3"/>
-    <!-- link 4 -->
-    <link name="${name}_link4">
+    <!-- Transmission 2 -->
+    <xacro:SimpleTransmission n="2" joint="${name}_joint_2"/>
+    <!-- link 3 -->
+    <link name="${name}_link_3">
       <collision>
         <origin xyz="0.01 0.06 0.01" rpy="0 ${pi/4} 0" />
@@ -195,8 +190,8 @@
       </inertial>
     </link>
-    <!-- Joint 4 -->
-    <joint name="${name}_joint4" type="revolute">
-      <parent link="${name}_link4"/>
-      <child link="${name}_link5"/>
+    <!-- Joint 3 -->
+    <joint name="${name}_joint_3" type="revolute">
+      <parent link="${name}_link_3"/>
+      <child link="${name}_link_4"/>
       <origin xyz="0.19500 0.0 0.03000" rpy="0 0 0"/>
       <axis xyz="1 0 0"/>
@@ -204,8 +199,8 @@
       <dynamics damping="0.7"/>
     </joint>
-    <!-- Transmission 4 -->
-    <xacro:SimpleTransmission n="4" joint="${name}_joint4"/>
-    <!-- link 5 -->
-    <link name="${name}_link5">
+    <!-- Transmission 3 -->
+    <xacro:SimpleTransmission n="3" joint="${name}_joint_3"/>
+    <!-- link 4 -->
+    <link name="${name}_link_4">
       <collision>
         <origin xyz="0.06 0 0.0" rpy="0 0 0" />
@@ -229,8 +224,8 @@
       </inertial>
     </link>
-    <!-- Joint 5 -->
-    <joint name="${name}_joint5" type="revolute">
-      <parent link="${name}_link5"/>
-      <child link="${name}_link6"/>
+    <!-- Joint 4 -->
+    <joint name="${name}_joint_4" type="revolute">
+      <parent link="${name}_link_4"/>
+      <child link="${name}_link_5"/>
       <origin xyz="0.06300 0.00 0.00000" rpy="0 0 0"/>
       <axis xyz="0 1 0"/>
@@ -238,8 +233,8 @@
       <dynamics damping="0.7"/>
     </joint>
-    <!-- Transmission 5 -->
-    <xacro:SimpleTransmission n="5" joint="${name}_joint5"/>
-    <!-- link 6 -->
-    <link name="${name}_link6">
+    <!-- Transmission 4 -->
+    <xacro:SimpleTransmission n="4" joint="${name}_joint_4"/>
+    <!-- link 5 -->
+    <link name="${name}_link_5">
       <collision>
         <origin xyz="0.005 0.045 0.0" rpy="0 0 0" />
@@ -281,7 +276,7 @@
       </inertial>
     </link>
-    <!-- Joint 6 -->
-    <joint name="${name}_joint6" type="revolute">
-      <parent link="${name}_link6"/>
+    <!-- Joint 5 -->
+    <joint name="${name}_joint_5" type="revolute">
+      <parent link="${name}_link_5"/>
       <child link="${name}_end_link"/>
       <origin xyz="0.12300 0.000 0.00000" rpy="0 0 0"/>
@@ -290,6 +285,6 @@
       <dynamics damping="0.7"/>
     </joint>
-    <!-- Transmission 6 -->
-    <xacro:SimpleTransmission n="6" joint="${name}_joint6"/>
+    <!-- Transmission 5 -->
+    <xacro:SimpleTransmission n="5" joint="${name}_joint_5"/>
     <!-- end link -->
     <link name="${name}_end_link">
