Commit message: added proper collision geometry

File: open_manipulator_p_description/urdf/open_manipulator_p_macro.urdf.xacro (robot description, xacro)
@@ -34,7 +34,7 @@
     <link name="${name}_link1">
       <collision>
-        <origin xyz="0 0 0" rpy="0 0 0"/>
-        <geometry>
-          <mesh filename="package://open_manipulator_p_description/meshes/link_1.stl" scale="0.001 0.001 0.001"/>
+        <origin xyz="0 0 0.063" rpy="0 0 0" />
+        <geometry>
+          <box size="0.054 0.054 0.126" />
         </geometry>
       </collision>
@@ -67,7 +67,7 @@
     <link name="${name}_link2">
       <collision>
-        <origin xyz="0 0 0" rpy="0 0 0"/>
-        <geometry>
-          <mesh filename="package://open_manipulator_p_description/meshes/link_2.stl" scale="0.001 0.001 0.001"/>
+        <origin xyz="0 0 0.03" rpy="0 0 0" />
+        <geometry>
+          <box size="0.06 0.14 0.06" />
         </geometry>
       </collision>
@@ -101,7 +101,31 @@
     <link name="${name}_link3">
       <collision>
-        <origin xyz="0 0.069 0" rpy="0 0 0"/>
-        <geometry>
-          <mesh filename="package://open_manipulator_p_description/meshes/link_3.stl" scale="0.001 0.001 0.001"/>
+        <origin xyz="0.0 0.07 0.01" rpy="0 0 0" />
+        <geometry>
+          <box size="0.06 0.02 0.09" />
+        </geometry>
+      </collision>
+      <collision>
+        <origin xyz="0.0 -0.07 0.01" rpy="0 0 0" />
+        <geometry>
+          <box size="0.06 0.02 0.09" />
+        </geometry>
+      </collision>
+      <collision>
+        <origin xyz="0.0 0.0 0.045" rpy="0 0 0" />
+        <geometry>
+          <box size="0.06 0.16 0.02" />
+        </geometry>
+      </collision>
+      <collision>
+        <origin xyz="0.0 0.0 0.155" rpy="0 0 0" />
+        <geometry>
+          <box size="0.06 0.09 0.2" />
+        </geometry>
+      </collision>
+      <collision>
+        <origin xyz="0.025 0.0 0.26" rpy="0 ${pi/4} 0" />
+        <geometry>
+          <box size="0.07 0.115 0.08" />
         </geometry>
       </collision>
@@ -134,7 +158,25 @@
     <link name="${name}_link4">
       <collision>
-        <origin xyz="0 0.05750 0" rpy="0 0 0"/>
-        <geometry>
-          <mesh filename="package://open_manipulator_p_description/meshes/link_4.stl" scale="0.001 0.001 0.001"/>
+        <origin xyz="0.01 0.06 0.01" rpy="0 ${pi/4} 0" />
+        <geometry>
+          <box size="0.06 0.02 0.1" />
+        </geometry>
+      </collision>
+      <collision>
+        <origin xyz="0.01 -0.06 0.01" rpy="0 ${pi/4} 0" />
+        <geometry>
+          <box size="0.06 0.02 0.1" />
+        </geometry>
+      </collision>
+      <collision>
+        <origin xyz="0.13 0 0.03" rpy="0 0 0" />
+        <geometry>
+          <box size="0.2 0.09 0.06" />
+        </geometry>
+      </collision>
+      <collision>
+        <origin xyz="0.04 0 0.03" rpy="0 0 0" />
+        <geometry>
+          <box size="0.03 0.14 0.06" />
         </geometry>
       </collision>
@@ -167,7 +209,7 @@
     <link name="${name}_link5">
       <collision>
-        <origin xyz="0 0 0" rpy="0 0 0"/>
-        <geometry>
-          <mesh filename="package://open_manipulator_p_description/meshes/link_5.stl" scale="0.001 0.001 0.001"/>
+        <origin xyz="0.06 0 0.0" rpy="0 0 0" />
+        <geometry>
+          <box size="0.055 0.09 0.05" />
         </geometry>
       </collision>
@@ -201,7 +243,25 @@
     <link name="${name}_link6">
       <collision>
-        <origin xyz="0 0.04500 0" rpy="0 0 0"/>
-        <geometry>
-          <mesh filename="package://open_manipulator_p_description/meshes/link_6.stl" scale="0.001 0.001 0.001"/>
+        <origin xyz="0.005 0.045 0.0" rpy="0 0 0" />
+        <geometry>
+          <box size="0.07 0.015 0.05" />
+        </geometry>
+      </collision>
+      <collision>
+        <origin xyz="0.005 -0.045 0.0" rpy="0 0 0" />
+        <geometry>
+          <box size="0.07 0.015 0.05" />
+        </geometry>
+      </collision>
+      <collision>
+        <origin xyz="0.035 0.0 0.0" rpy="0 0 0" />
+        <geometry>
+          <box size="0.02 0.105 0.05" />
+        </geometry>
+      </collision>
+      <collision>
+        <origin xyz="0.08 0.0 0.0" rpy="0 0 0" />
+        <geometry>
+          <box size="0.09 0.045 0.045" />
         </geometry>
       </collision>
@@ -235,7 +295,7 @@
     <link name="${name}_end_link">
       <collision>
-        <origin xyz="0 0 0" rpy="0 0 0"/>
-        <geometry>
-          <mesh filename="package://open_manipulator_p_description/meshes/end_link.stl" scale="0.001 0.001 0.001"/>
+        <origin xyz="0.01 0.0 0.0" rpy="0 0 0" />
+        <geometry>
+          <box size="0.02 0.06 0.045" />
         </geometry>
       </collision>

Commit message: improved the arm joint limits

File: open_manipulator_p_description/urdf/open_manipulator_p_macro.urdf.xacro (robot description, xacro)
@@ -54,5 +54,5 @@
       <origin xyz="0.0 0.0 0.126" rpy="0 0 0"/>
       <axis xyz="0 0 1"/>
-      <limit velocity="6.5" effort="1000" lower="${-pi*0.5}" upper="${pi*0.5}"/>
+      <limit velocity="6.5" effort="1000" lower="${-178 * pi/180}" upper="${178 * pi/180}"/>
       <dynamics damping="0.7"/>
     </joint>
@@ -88,5 +88,5 @@
       <origin xyz="0.0 0.0 0.033" rpy="0 0 0"/>
       <axis xyz="0 1 0"/>
-      <limit velocity="6.5" effort="1000" lower="${-pi*0.5}" upper="${pi*0.5}"/>
+      <limit velocity="6.5" effort="1000" lower="${-104 * pi/180}" upper="${104 * pi/180}"/>
       <dynamics damping="0.7"/>
     </joint>
@@ -145,5 +145,5 @@
       <origin xyz="0.03000 0.0 0.26400" rpy="0 0 0"/>
       <axis xyz="0 1 0"/>
-      <limit velocity="6.5" effort="1000" lower="${-pi*0.5}" upper="${pi*0.5}"/>
+      <limit velocity="6.5" effort="1000" lower="${-124 * pi/180}" upper="${85 * pi/180}"/>
       <dynamics damping="0.7"/>
     </joint>
@@ -196,5 +196,5 @@
       <origin xyz="0.19500 0.0 0.03000" rpy="0 0 0"/>
       <axis xyz="1 0 0"/>
-      <limit velocity="6.5" effort="1000" lower="${-pi*0.5}" upper="${pi*0.5}"/>
+      <limit velocity="6.5" effort="1000" lower="${-178 * pi/180}" upper="${178 * pi/180}"/>
       <dynamics damping="0.7"/>
     </joint>
@@ -230,5 +230,5 @@
       <origin xyz="0.06300 0.00 0.00000" rpy="0 0 0"/>
       <axis xyz="0 1 0"/>
-      <limit velocity="6.5" effort="1000" lower="${-pi*0.5}" upper="${pi*0.5}"/>
+      <limit velocity="6.5" effort="1000" lower="${-88 * pi/180}" upper="${88 * pi/180}"/>
       <dynamics damping="0.7"/>
     </joint>
@@ -282,5 +282,5 @@
       <origin xyz="0.12300 0.000 0.00000" rpy="0 0 0"/>
       <axis xyz="1 0 0"/>
-      <limit velocity="6.5" effort="1000" lower="${-pi*0.5}" upper="${pi*0.5}"/>
+      <limit velocity="6.5" effort="1000" lower="${-176 * pi/180}" upper="${176 * pi/180}"/>
       <dynamics damping="0.7"/>
     </joint>

Commit message: increased joint 4 limits

File: open_manipulator_p_description/urdf/open_manipulator_p_macro.urdf.xacro (robot description, xacro)
@@ -230,5 +230,5 @@
       <origin xyz="0.06300 0.00 0.00000" rpy="0 0 0"/>
       <axis xyz="0 1 0"/>
-      <limit velocity="6.5" effort="1000" lower="${-88 * pi/180}" upper="${88 * pi/180}"/>
+      <limit velocity="6.5" effort="1000" lower="${-95 * pi/180}" upper="${95 * pi/180}"/>
       <dynamics damping="0.7"/>
     </joint>

Commit message: reduced collision boxes for arm link 2

File: open_manipulator_p_description/urdf/open_manipulator_p_macro.urdf.xacro (robot description, xacro)
@@ -96,5 +96,5 @@
     <link name="${name}_link_2">
       <collision>
-        <origin xyz="0.0 0.07 0.01" rpy="0 0 0" />
+        <origin xyz="0.0 0.065 0.01" rpy="0 0 0" />
         <geometry>
           <box size="0.06 0.02 0.09" />
@@ -102,5 +102,5 @@
       </collision>
       <collision>
-        <origin xyz="0.0 -0.07 0.01" rpy="0 0 0" />
+        <origin xyz="0.0 -0.065 0.01" rpy="0 0 0" />
         <geometry>
           <box size="0.06 0.02 0.09" />
@@ -110,5 +110,5 @@
         <origin xyz="0.0 0.0 0.045" rpy="0 0 0" />
         <geometry>
-          <box size="0.06 0.16 0.02" />
+          <box size="0.06 0.15 0.02" />
         </geometry>
       </collision>

Commit message: optimized ellbow collision geometry

File: open_manipulator_p_description/urdf/open_manipulator_p_macro.urdf.xacro (robot description, xacro)
@@ -120,7 +120,13 @@
       </collision>
       <collision>
-        <origin xyz="0.025 0.0 0.26" rpy="0 ${pi/4} 0" />
-        <geometry>
-          <box size="0.07 0.115 0.08" />
+        <origin xyz="0.03 0.0 0.26" rpy="0 ${pi/4} 0" />
+        <geometry>
+          <box size="0.06 0.115 0.06" />
+        </geometry>
+      </collision>
+      <collision>
+        <origin xyz="-0.01 0.0 0.27" rpy="0 ${pi/4} 0" />
+        <geometry>
+          <box size="0.01 0.07 0.04" />
         </geometry>
       </collision>
@@ -153,13 +159,13 @@
     <link name="${name}_link_3">
       <collision>
-        <origin xyz="0.01 0.06 0.01" rpy="0 ${pi/4} 0" />
-        <geometry>
-          <box size="0.06 0.02 0.1" />
-        </geometry>
-      </collision>
-      <collision>
-        <origin xyz="0.01 -0.06 0.01" rpy="0 ${pi/4} 0" />
-        <geometry>
-          <box size="0.06 0.02 0.1" />
+        <origin xyz="0.015 0.06 0.015" rpy="0 ${pi/4} 0" />
+        <geometry>
+          <box size="0.05 0.02 0.08" />
+        </geometry>
+      </collision>
+      <collision>
+        <origin xyz="0.015 -0.06 0.015" rpy="0 ${pi/4} 0" />
+        <geometry>
+          <box size="0.05 0.02 0.08" />
         </geometry>
       </collision>

Commit message: adjusted joint limits

File: open_manipulator_p_description/urdf/open_manipulator_p_macro.urdf.xacro (robot description, xacro)
@@ -54,5 +54,5 @@
       <origin xyz="0.0 0.0 0.126" rpy="0 0 0"/>
       <axis xyz="0 0 1"/>
-      <limit velocity="6.5" effort="1000" lower="${-178 * pi/180}" upper="${178 * pi/180}"/>
+      <limit velocity="6.5" effort="1000" lower="-2" upper="2.1"/>
       <dynamics damping="0.7"/>
     </joint>
@@ -88,5 +88,5 @@
       <origin xyz="0.0 0.0 0.033" rpy="0 0 0"/>
       <axis xyz="0 1 0"/>
-      <limit velocity="6.5" effort="1000" lower="${-104 * pi/180}" upper="${104 * pi/180}"/>
+      <limit velocity="6.5" effort="1000" lower="-1.5" upper="1.4"/>
       <dynamics damping="0.7"/>
     </joint>
@@ -202,5 +202,5 @@
       <origin xyz="0.19500 0.0 0.03000" rpy="0 0 0"/>
       <axis xyz="1 0 0"/>
-      <limit velocity="6.5" effort="1000" lower="${-178 * pi/180}" upper="${178 * pi/180}"/>
+      <limit velocity="6.5" effort="1000" lower="-2.9" upper="2.85"/>
       <dynamics damping="0.7"/>
     </joint>

Commit message: new arm limits

File: open_manipulator_p_description/urdf/open_manipulator_p_macro.urdf.xacro (robot description, xacro)
@@ -288,5 +288,5 @@
       <origin xyz="0.12300 0.000 0.00000" rpy="0 0 0"/>
       <axis xyz="1 0 0"/>
-      <limit velocity="6.5" effort="1000" lower="${-176 * pi/180}" upper="${176 * pi/180}"/>
+      <limit velocity="6.5" effort="1000" lower="${-174 * pi/180}" upper="${174 * pi/180}"/>
       <dynamics damping="0.7"/>
     </joint>

Commit message: reduced joint 5 joint range

File: open_manipulator_p_description/urdf/open_manipulator_p_macro.urdf.xacro (robot description, xacro)
@@ -288,5 +288,5 @@
       <origin xyz="0.12300 0.000 0.00000" rpy="0 0 0"/>
       <axis xyz="1 0 0"/>
-      <limit velocity="6.5" effort="1000" lower="${-174 * pi/180}" upper="${174 * pi/180}"/>
+      <limit velocity="6.5" effort="1000" lower="${-174 * pi/180}" upper="${159 * pi/180}"/>
       <dynamics damping="0.7"/>
     </joint>

Commit message: Reduced joint effort to match max current of real servos

File: open_manipulator_p_description/urdf/open_manipulator_p_macro.urdf.xacro (robot description, xacro)
@@ -54,5 +54,5 @@
       <origin xyz="0.0 0.0 0.126" rpy="0 0 0"/>
       <axis xyz="0 0 1"/>
-      <limit velocity="6.5" effort="1000" lower="-2" upper="2.1"/>
+      <limit velocity="6.5" effort="10" lower="-2" upper="2.1"/>
       <dynamics damping="0.7"/>
     </joint>
@@ -88,5 +88,5 @@
       <origin xyz="0.0 0.0 0.033" rpy="0 0 0"/>
       <axis xyz="0 1 0"/>
-      <limit velocity="6.5" effort="1000" lower="-1.5" upper="1.4"/>
+      <limit velocity="6.5" effort="10" lower="-1.5" upper="1.4"/>
       <dynamics damping="0.7"/>
     </joint>
@@ -151,5 +151,5 @@
       <origin xyz="0.03000 0.0 0.26400" rpy="0 0 0"/>
       <axis xyz="0 1 0"/>
-      <limit velocity="6.5" effort="1000" lower="${-124 * pi/180}" upper="${85 * pi/180}"/>
+      <limit velocity="6.5" effort="10" lower="${-124 * pi/180}" upper="${85 * pi/180}"/>
       <dynamics damping="0.7"/>
     </joint>
@@ -202,5 +202,5 @@
       <origin xyz="0.19500 0.0 0.03000" rpy="0 0 0"/>
       <axis xyz="1 0 0"/>
-      <limit velocity="6.5" effort="1000" lower="-2.9" upper="2.85"/>
+      <limit velocity="6.5" effort="10" lower="-2.9" upper="2.85"/>
       <dynamics damping="0.7"/>
     </joint>
@@ -236,5 +236,5 @@
       <origin xyz="0.06300 0.00 0.00000" rpy="0 0 0"/>
       <axis xyz="0 1 0"/>
-      <limit velocity="6.5" effort="1000" lower="${-95 * pi/180}" upper="${95 * pi/180}"/>
+      <limit velocity="6.5" effort="10" lower="${-95 * pi/180}" upper="${95 * pi/180}"/>
       <dynamics damping="0.7"/>
     </joint>
@@ -288,5 +288,5 @@
       <origin xyz="0.12300 0.000 0.00000" rpy="0 0 0"/>
       <axis xyz="1 0 0"/>
-      <limit velocity="6.5" effort="1000" lower="${-174 * pi/180}" upper="${159 * pi/180}"/>
+      <limit velocity="6.5" effort="10" lower="${-174 * pi/180}" upper="${159 * pi/180}"/>
       <dynamics damping="0.7"/>
     </joint>

Commit message: Added optional geometry for depth filtering

File: open_manipulator_p_description/urdf/open_manipulator_p_macro.urdf.xacro (robot description, xacro)
@@ -21,4 +21,5 @@
   <xacro:macro name="open_manipulator_p_macro" params="name parent *origin">
     <xacro:open_manipulator_p_gazebo_macro name="${name}"/>
+    <xacro:arg name="use_depth_self_filter" default="true"/>
     <joint name="${name}_fixed_joint" type="fixed">
       <xacro:insert_block name="origin"/>
@@ -144,4 +145,19 @@
         <!--<inertia ixx="0.01111021" ixy="0.00001331" ixz="-0.00134208" iyy="0.01046642" iyz="0.00016235" izz="0.00202081" />-->
       </inertial>
+      <!-- Depth Self Filter box -->
+      <xacro:if value="$(arg use_depth_self_filter)">
+        <collision>
+          <origin xyz="0.0 0.0 0.1" rpy="0 0 0" />
+          <geometry>
+            <box size="0.1 0.1 0.35" />
+          </geometry>
+        </collision>
+        <collision>
+          <origin xyz="0.0 0.0 0.0" rpy="0 0 0" />
+          <geometry>
+            <box size="0.18 0.18 0.17" />
+          </geometry>
+        </collision>
+      </xacro:if>
     </link>
     <!-- Joint 2 -->
@@ -195,4 +211,31 @@
         <!--<inertia ixx="0.00096726" ixy="0.00004383" ixz="-0.00002771" iyy="0.00318801" iyz="0.00000627" izz="0.00341484" />-->
       </inertial>
+      <!-- Depth Self Filter box -->
+      <xacro:if value="$(arg use_depth_self_filter)">
+        <collision>
+          <origin xyz="-0.02 0.0 0.02" rpy="${pi/2} 0 0" />
+          <geometry>
+            <cylinder radius="0.07" length="0.20"/>
+          </geometry>
+        </collision>
+        <collision>
+          <origin xyz="-0.02 0.04 0.02" rpy="${pi/2} 0 0" />
+          <geometry>
+            <cylinder radius="0.1" length="0.12"/>
+          </geometry>
+        </collision>
+        <!--<collision>
+          <origin xyz="0.17 0.0 0.0" rpy="0 ${pi/2} 0" />
+          <geometry>
+            <cylinder radius="0.1" length="0.35"/>
+          </geometry>
+        </collision>-->
+        <collision>
+          <origin xyz="0.17 0.01 0.02" rpy="0 0 0" />
+          <geometry>
+            <box size="0.35 0.16 0.16" />
+          </geometry>
+        </collision>
+      </xacro:if>
     </link>
     <!-- Joint 3 -->
@@ -229,4 +272,13 @@
         <!--<inertia ixx="0.00030285" ixy="0.00000761" ixz="0.00000031" iyy="0.00022339" iyz="-0.00000001" izz="0.00039766" />-->
       </inertial>
+      <!-- Depth Self Filter box -->
+      <xacro:if value="$(arg use_depth_self_filter)">
+        <collision>
+          <origin xyz="0.08 0.0 0.0" rpy="0 0 0" />
+          <geometry>
+            <sphere radius="0.11"/>
+          </geometry>
+        </collision>
+      </xacro:if>
     </link>
     <!-- Joint 4 -->
@@ -281,4 +333,13 @@
         <!--<inertia ixx="0.00021512" ixy="0.00001009" ixz="0.00000000" iyy="0.00042827" iyz="0.00000000" izz="0.00051436" />-->
       </inertial>
+      <!-- Depth Self Filter box
+      <xacro:if value="$(arg use_depth_self_filter)">
+        <collision>
+          <origin xyz="0.03 0.0 -0.01" rpy="0 0 0" />
+          <geometry>
+            <box size="0.18 0.135 0.15" />
+          </geometry>
+        </collision>
+      </xacro:if> -->
     </link>
     <!-- Joint 5 -->
@@ -295,4 +356,13 @@
     <!-- end link -->
     <link name="${name}_end_link">
+      <!-- Depth Self Filter box-->
+      <xacro:if value="$(arg use_depth_self_filter)">
+        <collision>
+          <origin xyz="0.05 0.0 0.0" rpy="0 ${pi/2} 0" />
+          <geometry>
+            <cylinder radius="0.10" length="0.23"/>
+          </geometry>
+        </collision>
+      </xacro:if>
       <collision>
         <origin xyz="0.01 0.0 0.0" rpy="0 0 0" />

Commit message: remove unused geometry and renamed param to use_depth_filter_geometry

File: open_manipulator_p_description/urdf/open_manipulator_p_macro.urdf.xacro (robot description, xacro)
@@ -21,5 +21,5 @@
   <xacro:macro name="open_manipulator_p_macro" params="name parent *origin">
     <xacro:open_manipulator_p_gazebo_macro name="${name}"/>
-    <xacro:arg name="use_depth_self_filter" default="false"/>
+    <xacro:arg name="use_depth_filter_geometry" default="false"/>
     <joint name="${name}_fixed_joint" type="fixed">
       <xacro:insert_block name="origin"/>
@@ -145,6 +145,6 @@
         <!--<inertia ixx="0.01111021" ixy="0.00001331" ixz="-0.00134208" iyy="0.01046642" iyz="0.00016235" izz="0.00202081" />-->
       </inertial>
-      <!-- Depth Self Filter box -->
-      <xacro:if value="$(arg use_depth_self_filter)">
+      <!-- Depth Filter Geometry -->
+      <xacro:if value="$(arg use_depth_filter_geometry)">
         <collision>
           <origin xyz="0.0 0.0 0.1" rpy="0 0 0" />
@@ -211,6 +211,6 @@
         <!--<inertia ixx="0.00096726" ixy="0.00004383" ixz="-0.00002771" iyy="0.00318801" iyz="0.00000627" izz="0.00341484" />-->
       </inertial>
-      <!-- Depth Self Filter box -->
-      <xacro:if value="$(arg use_depth_self_filter)">
+      <!-- Depth Filter Geometry -->
+      <xacro:if value="$(arg use_depth_filter_geometry)">
         <collision>
           <origin xyz="-0.02 0.0 0.02" rpy="${pi/2} 0 0" />
@@ -225,10 +225,4 @@
           </geometry>
         </collision>
-        <!--<collision>
-          <origin xyz="0.17 0.0 0.0" rpy="0 ${pi/2} 0" />
-          <geometry>
-            <cylinder radius="0.1" length="0.35"/>
-          </geometry>
-        </collision>-->
         <collision>
           <origin xyz="0.17 0.01 0.02" rpy="0 0 0" />
@@ -272,6 +266,6 @@
         <!--<inertia ixx="0.00030285" ixy="0.00000761" ixz="0.00000031" iyy="0.00022339" iyz="-0.00000001" izz="0.00039766" />-->
       </inertial>
-      <!-- Depth Self Filter box -->
-      <xacro:if value="$(arg use_depth_self_filter)">
+      <!-- Depth Filter Geometry -->
+      <xacro:if value="$(arg use_depth_filter_geometry)">
         <collision>
           <origin xyz="0.08 0.0 0.0" rpy="0 0 0" />
@@ -333,13 +327,4 @@
         <!--<inertia ixx="0.00021512" ixy="0.00001009" ixz="0.00000000" iyy="0.00042827" iyz="0.00000000" izz="0.00051436" />-->
       </inertial>
-      <!-- Depth Self Filter box
-      <xacro:if value="$(arg use_depth_self_filter)">
-        <collision>
-          <origin xyz="0.03 0.0 -0.01" rpy="0 0 0" />
-          <geometry>
-            <box size="0.18 0.135 0.15" />
-          </geometry>
-        </collision>
-      </xacro:if> -->
     </link>
     <!-- Joint 5 -->
@@ -356,6 +341,6 @@
     <!-- end link -->
     <link name="${name}_end_link">
-      <!-- Depth Self Filter box-->
-      <xacro:if value="$(arg use_depth_self_filter)">
+      <!-- Depth Filter Geometry -->
+      <xacro:if value="$(arg use_depth_filter_geometry)">
         <collision>
           <origin xyz="0.05 0.0 0.0" rpy="0 ${pi/2} 0" />
